File: keystone-esp/keystone-esp.kicad_pcb (KiCad board)
At the start: 2 copper layers, 46 x 41 mm, 40 parts, among them J1 USBC_TH_2, J2 Conn_01x06_Socket, J3 Conn_01x12_Socket, J4 Conn_01x15_Socket, Q1 BSS138, Q2 BSS138, Q3 AO3400A, Q4 AO3400A, SW1 SW_Push, U1 SN74AHC1G14DBVR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

Commit message: Blurp murp squiggle eeo eeo rrrrr
Parts:
- added TP1: TestPoint, TestPoint:TestPoint_Pad_D1.5mm, B.Cu at (187.1, 99.6)
- added TP10: TestPoint, TestPoint:TestPoint_Pad_D1.5mm, B.Cu at (213.7, 86.2)
- added TP11: TestPoint, TestPoint:TestPoint_Pad_D1.5mm, B.Cu at (212.5, 107.4)
- added TP12: TestPoint, TestPoint:TestPoint_Pad_D1.5mm, B.Cu at (216.0, 105.8)
- added TP2: TestPoint, TestPoint:TestPoint_Pad_D1.5mm, B.Cu at (186.7, 94.5)
- added TP3: TestPoint, TestPoint:TestPoint_Pad_D1.5mm, B.Cu at (185.2, 97.5)
- added TP4: TestPoint, TestPoint:TestPoint_Pad_D1.5mm, B.Cu at (196.1, 99.8)
- added TP5: TestPoint, TestPoint:TestPoint_Pad_D1.5mm, B.Cu at (205.4, 101.2)
- added TP6: TestPoint, TestPoint:TestPoint_Pad_D1.5mm, B.Cu at (207.8, 96.9)
- added TP7: TestPoint, TestPoint:TestPoint_Pad_D1.5mm, B.Cu at (193.7, 90.3)
- added TP8: TestPoint, TestPoint:TestPoint_Pad_D1.5mm, B.Cu at (203.1, 105.5)
- added TP9: TestPoint, TestPoint:TestPoint_Pad_D1.5mm, B.Cu at (185.7, 79.0)
- moved REF** 20.8 mm to (182.1, 84.7), turned to 90 degrees
- moved FID2 13.9 mm to (184.9, 90.4)
- moved R10 5.11 mm to (185.8, 82.4)
- moved SW1 2.99 mm to (185.9, 78.4)
- moved FID1 1.44 mm to (179.7, 78.4)
- turned JP3 to 180 degrees
Routing:
- net GND: track 28.6 -> 40.8 mm, vias 15 -> 17
- net /IO22: track 12.9 -> 22.5 mm
- net /EN: track 78.0 -> 84.9 mm
- net VCC: track 148.0 -> 144.4 mm, vias 5 -> 6
- net /IO0: track 57.5 -> 59.3 mm
- net /RX: track 64.7 -> 66.1 mm
- net Net-(JP3-B): track 4.04 -> 5.40 mm
- net /TX: track 61.9 -> 63.2 mm
- net Net-(J1-CC2): track 13.1 -> 14.1 mm, vias 0 -> 1
- net Net-(J1-CC1): track 3.87 -> 4.64 mm, vias 0 -> 1
- net /IO21: track 10.7 -> 11.3 mm, vias 0 -> 1
- net Net-(J1-DP1): track 27.2 -> 27.3 mm, vias 0 -> 1
Other:
- board text added: "-ESP"
- board text added: "13"
- board text added: "14"
- board text added: "15"
- board text added: "16"
- board text added: "17"
- board text added: "18"
- board text added: "19"
- board text added: "21"
- board text added: "22"
- board text added: "23"
- board text added: "25"
- board text added: "26"
- board text added: "27"
- board text added: "32"
- board text added: "33"
- board text added: "34"
- board text added: "35"
- board text added: "36"
- board text added: "39"
- board text added: "4"
- board text added: "5"
- board text added: "GND"
- board text added: "VCC"
- board text added: "V_BUS"
- board text added: "by RobotZwrrl.xyz RobotMissions.org 04-09-24 v1.2"
- board text added: "keystone-esp"
- board text removed: "by RobotZwrrl.xyz RobotMissions.org 03-09-24 v1.1"
