File: keystone-esp/keystone-esp.kicad_sch (KiCad schematic)
At the start: 39 parts, among them J1 USBC_TH_2, J2 Conn_01x06_Socket, J3 Conn_01x12_Socket, J4 Conn_01x15_Socket, Q1 BSS138, Q2 BSS138, Q3 AO3400A, Q4 AO3400A, SW1 SW_Push, U1 SN74AHC1G14DBVR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

Commit message: Blurp murp squiggle eeo eeo rrrrr
Parts:
- added TP1, TP10, TP11, TP12, TP2, TP3, TP4, TP5, TP6, TP7, TP8, TP9: TestPoint, TestPoint:TestPoint_Pad_D1.5mm, symbol Connector:TestPoint
- C3: Digikey 1276-3179-1-ND -> 399-C1206C475K5RAC7800CT-ND; Digikey2 (none) -> 1276-3179-1-ND
- D1, D2, D3: Digikey 160-1170-1-ND -> 160-1406-1-ND
- R10, R6, R9: Digikey 311-10.0KFRCT-ND -> RMCF1206FT10K0CT-ND; Digikey2 (none) -> 311-10.0KFRCT-ND
- R3, R4, R5: value 1k -> 330; Digikey 311-1.00KFRCT-ND -> RMCF1206FT330RCT-ND; Digikey2 (none) -> 311-330FRCT-ND
- R7, R8: Digikey 311-4.70KFRCT-ND -> RMCF1206FT4K70CT-ND; Digikey2 (none) -> 311-4.70KFRCT-ND
Connections:
- net EN: now also TP7.1
- net GND: now also TP10.1
- net IO0: now also TP8.1
- net IO21: now also TP11.1
- net IO22: now also TP12.1
- net RX: now also TP5.1
- net TX: now also TP6.1
- net VCC: now also TP9.1
- net at J1.A5 (CC1), R2.1: now also TP2.1
- net at J1.A6 (DP1), J1.B6 (DP2), U2.5 (UD+): now also TP4.1
- net at J1.A7 (DN1), J1.B7 (DN2), U2.6 (UD-): now also TP3.1
- net at J1.B5 (CC2), R1.1: now also TP1.1
Other:
- note added: "Boostlet!'s 3.3V output is connected to Keystone's VCC input"
- note added: "Keystone (C) Copyright Erin RobotZwrrl, Robot Missions Inc. 04-09-24 v1.2 RobotZwrrl.xyz/boostlet RobotMissions.org This hardware is released under: CERN Open Hardware License Version 2.0 - Permissive (CERN-OHL-P) Disclaimer: Distributed as is. No warranty is given. Not responsible or liable for any damage or harm that result from this product."
- note added: "LEDs - RX/TX"
- note added: "RX/TX is active low, so using an inverter to make the LEDs light up on data transmission"
- note removed: "Boostlet!'s 3.3V output is connected to Keystone's VCC"
- note removed: "Keystone (C) Copyright Erin RobotZwrrl, Robot Missions Inc. 03-09-24 v1.1 RobotZwrrl.xyz/boostlet RobotMissions.org This hardware is released under: CERN Open Hardware License Version 2.0 - Permissive (CERN-OHL-P) Disclaimer: Distributed as is. No warranty is given. Not responsible or liable for any damage or harm that result from this product."
- note removed: "LEDs - TX/RX"
- note removed: "Programming header"
- moved on the sheet: C1, C2, C3, C4, C5, C6, D3, J1, J2, J3, J4, JP1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
